Commit message: Implemented remote control and SLAM autonomous navigation

File: src/mybot_description/urdf/mybot.xacro (robot description, xacro)
@@ -12,12 +12,12 @@
       <origin xyz="0 0.3 0" rpy=" 0 0 0"/>
       <inertia
-          ixx="1.0" ixy="0" ixz="0"
-          iyy="1.0" iyz="0"
-          izz="1.0"
+          ixx="0.1" ixy="0" ixz="0"
+          iyy="0.1" iyz="0"
+          izz="0.1"
       />
     </inertial>
     <collision name='collision'>
      <geometry>
-        <box size="1 1.5 0.2"/>
+        <box size=".8 1.2 0.15"/>
       </geometry>
     </collision>
@@ -25,12 +25,12 @@
       <origin xyz="0 0 0" rpy=" 0 0 0"/>
      <geometry>
-        <box size="1 1.5 0.2"/>
+        <box size=".8 1.2 0.15"/>
       </geometry>
     </visual>
 <!-- -->
     <collision name='caster_collision1'>
-      <origin xyz="0 -0.5 -0.1" rpy=" 0 0 0"/>
+      <origin xyz="0 -0.4 -0.1" rpy=" 0 0 0"/>
       <geometry>
-        <sphere radius="0.2"/>
+        <sphere radius="0.15"/>
       </geometry>
       <surface>
@@ -46,13 +46,13 @@
     </collision>
     <visual name='caster_visual1'>
-      <origin xyz="0 -0.5 -0.1" rpy=" 0 0 0"/>
+      <origin xyz="0 -0.4 -0.1" rpy=" 0 0 0"/>
       <geometry>
-        <sphere radius="0.2"/>
+        <sphere radius="0.15"/>
       </geometry>
     </visual>
     <collision name='caster_collision2'>
-      <origin xyz="0 0.5 -0.1" rpy=" 0 0 0"/>
+      <origin xyz="0 0.4 -0.1" rpy=" 0 0 0"/>
       <geometry>
-        <sphere radius="0.2"/>
+        <sphere radius="0.15"/>
       </geometry>
       <surface>
@@ -68,7 +68,7 @@
     </collision>
     <visual name='caster_visual2'>
-      <origin xyz="0 0.5 -0.1" rpy=" 0 0 0"/>
+      <origin xyz="0 0.4 -0.1" rpy=" 0 0 0"/>
       <geometry>
-        <sphere radius="0.2"/>
+        <sphere radius="0.15"/>
       </geometry>
     </visual>
@@ -129,5 +129,5 @@
     <axis xyz="1 0 0" rpy="0 0 0"/>
     <limit effort="100" velocity="100"/>
-    <joint_properties damping="0.0" friction="0.0"/>
+    <joint_properties damping="1.0" friction="1.0"/>
   </joint>
   <joint type="continuous" name="right_wheel_hinge">
@@ -138,5 +138,5 @@
     <axis xyz="1 0 0" rpy="0 0 0"/>
     <limit effort="100" velocity="100"/>
-    <joint_properties damping="0.0" friction="0.0"/>
+    <joint_properties damping="1.0" friction="1.0"/>
   </joint>
 <!--   camera  -->
